Commit message: tip/ add hand

File: URDF/mega_robot_1st_urdf/urdf/whole_robot_moveit.urdf (robot description, URDF)
Before this commit: robot mega_robot_1st_urdf, 22 links, 21 joints
Links:
- added link left_tool; collision box size=0.001 0.001 0.001; visual box size=0.001 0.001 0.001
- added link right_tool; collision box size=0.001 0.001 0.001; visual box size=0.001 0.001 0.001
Joints:
- added joint left_tool_joint: type fixed, parent lhand, child left_tool, origin xyz=0 0 0 rpy=-2.541592653589793 0 2.7707963267948967
- added joint right_tool_joint: type fixed, parent rhand, child right_tool, origin xyz=0 0 0 rpy=2.541592653589793 0 2.7707963267948967
